File: AK4490DAC.kicad_sch (KiCad schematic)
At the start: 82 parts, among them IC1 LP5907MFX-3.3/NOPB, IC2 LP5907MFX-3.3/NOPB, IC3 LP5907MFX-3.3/NOPB, IC4 TPS7A2050PDBVR, IC5 MUSES8920, IC8 TPS7A2050PDBVR, IC9 AMS1117, J1 JST_XA_B02B-XASK-1, J2 USB_C_Receptacle_USB2.0_16P, J3 TORX147FT, J4 LINE_OUT_L, J5 LINE_OUT_R, T1 DA103C, U1 SN74LS06NSR, U2 PCM2704CDBR, U3 TCM809TENB713, U4 TCM809TENB713, U5 AK4118, U6 AK4490, U7 MCWI03-12D15, Y1 11.2896MHz, Y2 12MHz

Commit message: Remove PCM2704C, AK4118 and SPDIF path ahead of XU316 migration
Per user decision to replace both PCM2704C (USB audio) and AK4118
(SPDIF receiver) with a single XU316-1024-QF60B-C24 (XMOS xCORE.ai),
and to drop the optical SPDIF input entirely (USB-only device now):

Removed entirely (component + all exclusive support parts + wiring):
- U2 (PCM2704CDBR), Y2 (12MHz X'tal), R5/R6/R7 (USB D+/D- pullup/
  termination - not needed, XU316's USB PHY needs no external R per
  its datasheet's simplified reference diagram), C14-C20 (X'tal load
  caps + supply decoupling)
- U5 (AK4118), Y1 (11.2896MHz X'tal), R1 (pin39 pulldown), R10 (RX1
  termination), C1/C2 (X'tal load caps), C3 (VCOM cap), C5/C6/C7
  (AVDD/DVDD/TVDD decoupling)
- J3 (TORX147FT optical receiver), R2 (RX0 470R series), C4 (Vcc
  decoupling) - optical SPDIF input dropped per this session's decision
- JP1 (IPS0 RX0/RX1 select jumper) - meaningless without AK4118
- T1 (DA103C isolation transformer), R8 (DOUT series R), R9 (primary
  shunt), C21 (secondary DC block) - this was the galvanic isolation
  path between PCM2704C's USB-side ground and AK4118's RX1; XU316
  driving AK4490's I2S directly eliminates this specific isolation
  mechanism (to be replaced by a USB-side isolator IC in a follow-up
  commit, per discussion)
- Orphaned lib_symbols cache entries: AK4490DAC:PCM2704CDBR,
  AK4490DAC:AK4118, AK4490DAC:TORX147FT, Transformer:TRANSF1,
  Connector_Generic:Conn_01x03 (JP1's symbol; Conn_01x02 stays, still
  used by J1/J4/J5)

Removal was done by paren-depth-bounded deletion of each component's
symbol block (30 components total), followed by two passes of removing
now-dangling stub wires/labels identified via kicad-cli sch erc's
unconnected_wire_endpoint/label_dangling violations (42 in the first
pass, 10 more that the first pass's removals exposed in a second pass) -
each removed by exact UUID match against the ERC report rather than by
coordinate, to avoid the coordinate-collision class of bug seen earli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
Parts:
- removed C1, C2: 18pF, Capacitor_SMD:C_0603_1608Metric, symbol Device:C
- removed C14, C15: 22pF, Capacitor_SMD:C_0603_1608Metric, symbol Device:C
- removed C16, C17, C18, C19: 1uF, Capacitor_SMD:C_0603_1608Metric, symbol Device:C
- removed C20: 10uF, Capacitor_SMD:C_0805_2012Metric, symbol Device:C
- removed C21, C4, C5, C6, C7: 0.1uF, Capacitor_SMD:C_0603_1608Metric, symbol Device:C
- removed C3: 0.47uF, Capacitor_SMD:C_0603_1608Metric, symbol Device:C
- removed J3: TORX147FT, AK4490DAC:TORX147FT, symbol AK4490DAC:TORX147FT
- removed JP1: IPS0_SEL, Connector_PinHeader_2.54mm:PinHeader_1x03_P2.54mm_Vertical, symbol Connector_Generic:Conn_01x03
- removed R1: 10k, Resistor_SMD:R_0603_1608Metric, symbol Device:R
- removed R10: 75, Resistor_SMD:R_0603_1608Metric, symbol Device:R
- removed R2: 470, Resistor_SMD:R_0603_1608Metric, symbol Device:R
- removed R5: 1.5k, Resistor_SMD:R_0603_1608Metric, symbol Device:R
- removed R6, R7: 22, Resistor_SMD:R_0603_1608Metric, symbol Device:R
- removed R8: 240, Resistor_SMD:R_0603_1608Metric, symbol Device:R
- removed R9: 120, Resistor_SMD:R_0603_1608Metric, symbol Device:R
- removed T1: DA103C, AK4490DAC:DA103C_MUR, symbol AK4490DAC:DA103C
- removed U2: PCM2704CDBR, Package_SO:SSOP-28_5.3x10.2mm_P0.65mm, symbol AK4490DAC:PCM2704CDBR
- removed U5: AK4118, Package_QFP:LQFP-48_7x7mm_P0.5mm, symbol AK4490DAC:AK4118
- removed Y1: 11.2896MHz, Crystal:Crystal_SMD_5032-2Pin_5.0x3.2mm, symbol Device:Crystal
- removed Y2: 12MHz, Crystal:Crystal_SMD_3225-4Pin_3.2x2.5mm, symbol Device:Crystal
Connections:
- net BICK: no longer names the net of U6.3 (BICK)
- net LRCK: no longer names the net of U6.5 (LRCK)
- net MCLK: no longer names the net of U6.46 (MCLK)
- net SDATA: no longer names the net of U6.4 (SDATA)
Other:
- moved on the sheet: C28, C29, C30, C31, J1, J2, R27, R28, U6

Commit message: Add XU316, ISOUSB211, QSPI flash: USB/SPDIF -> XMOS migration
Implements the XU316-1024-QF60B-C24 (XMOS xcore.ai) replacement for
PCM2704C+AK4118, decided and refined over several rounds of discussion
(power architecture, USB isolation approach and cost, GND domain
strategy). Firmware is explicitly out of scope - hardware only.

New parts:
- U2 = XU316-1024-QF60B-C24, custom 60-pin symbol (all pins present,
  named/typed per XMOS datasheet SLLSFC5D... er, XU316 datasheet
  section 3/4 pin tables) + custom parametric QFN-60 0.4mm-pitch
  footprint (dimensions estimated from the QF60B package designator -
  verify against the real mechanical drawing, including pin-1 corner
  orientation, before fab).
- U3 = ISOUSB211DPR (TI): USB isolator between J2/USB_GND (isolated,
  side1) and XU316/main GND (side2). Side1 bus-powered directly from
  J2's VBUS (both VBUS1 and VCC1 tied to it), so its internal LDOs
  generate V3P3V1/V1P8V1 locally - no separate isolated supply needed.
  Side2 uses external-supply mode from the new +3V3_XU/+1V8_XU rails.
  EQ1x/EQ2x tied to their GND (00 = shortest-trace default, verify
  against actual layout), CDPENZ1/2 tied high (disable CDP charging-port
  advertising, pure USB2.0 data only).
- U4 = W25Q32JVSSIQ: QSPI boot flash, wired per XU316 datasheet's boot
  pin table (X0D01=CS, X0D10=SCLK, X0D04/05/06/07=IO0-3).
- Y1 + C34/C35: 24MHz crystal per XU316's reference schematic (Figure
  2) - load cap value is a placeholder (18pF, matching this project's
  other crystals), verify against the chosen crystal's CL spec.
- IC10 (new, LP5907 1.8V) and IC11 (new, TPS7A20 ADJ variant + R29/R30
  divider targeting 0.9V) added for XU316's VDDIOB18/PLL_AVDD/USB_VDD18
  and VDD-core rails respectively. IC1 (previously AK4118's 3.3V LDO,
  now orphaned) repurposed as +3V3_XU. All three LDOs' EN tied to IN
  (always-on); IN itself is left for the user's main power wiring pass,
  consistent with how IC2-4/8/9 were already left.
- JP2: 5-pin JTAG debug heade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
Parts:
- added C34, C35: 18pF, Capacitor_SMD:C_0603_1608Metric, symbol Device:C
- added IC10: LP5907MFX-1.8, Package_TO_SOT_SMD:SOT-23-5, symbol Regulator_Linear:LP5907MFX-3.3
- added IC11: TPS7A20-ADJ, Package_TO_SOT_SMD:SOT-23-5, symbol AK4490DAC:TPS7A2050PDBVR
- added JP2: JTAG_DEBUG, Connector_PinHeader_2.54mm:PinHeader_1x05_P2.54mm_Vertical, symbol Connector_Generic:Conn_01x05
- added R29: 1.2k, Resistor_SMD:R_0603_1608Metric, symbol Device:R
- added R30: 10k, Resistor_SMD:R_0603_1608Metric, symbol Device:R
- added U2: XU316-1024-QF60B-C24, AK4490DAC:XU316_QF60B_7x7, symbol AK4490DAC:XU316-1024-QF60B-C24
- added U3: ISOUSB211DPR, Package_SO:SSOP-28_5.3x10.2mm_P0.65mm, symbol AK4490DAC:ISOUSB211
- added U4: W25Q32JVSSIQ, Package_SO:SOIC-8_3.9x4.9mm_P1.27mm, symbol AK4490DAC:W25Q32JVSSIQ
- added Y1: 24MHz, Crystal:Crystal_SMD_3225-4Pin_3.2x2.5mm, symbol Device:Crystal
Connections:
- net GND: now also IC1.2 (GND), C34.2, C35.2, IC10.2 (GND), IC11.2 (GND), JP2.5 (Pin_5), R30.2, U2.65 (VSS_EP), U3.17 (GND2_B), U3.19 (EQ21), U3.20 (EQ20), U3.26 (GND2), U4.4 (GND)
- net USB_D+: now also U3.8 (UD+)
- net USB_D-: now also U3.7 (UD-)
- net USB_GND: now also U3.10 (EQ11), U3.12 (GND1_B), U3.3 (GND1), U3.9 (EQ10)
- net VBUS: now also U3.1 (VBUS1), U3.13 (CDPENZ1), U3.5 (VCC1)
- net BICK: now reaches U6.3 (BICK)
- net BICK: now also U2.9 (X1D00_BICK)
- net SDATA: now reaches U6.4 (SDATA)
- net SDATA: now also U2.13 (X1D10_SDATA)
- net MCLK: now reaches U6.46 (MCLK)
- net MCLK: now also U2.14 (X1D11_MCLK)
- net LRCK: now reaches U6.5 (LRCK)
- net LRCK: now also U2.10 (X1D01_LRCK)
- net at IC1.1 (IN): now also IC1.3 (EN)
- net +3V3_XU: now reaches IC1.5 (OUT)
- net +3V3_XU: now also U2.30 (USB_VDD33), U2.38 (VDDIOR), U2.52 (VDDIOT), U2.8 (VDDIOL), U3.16 (CDPENZ2), U3.27 (V3P3V2), U3.28 (VBUS2), U4.8 (VCC)
- new net: IC11.1 (IN), IC11.3 (EN)
- new net: IC10.1 (IN), IC10.3 (EN)
- new net +0V9_XU: IC11.5 (OUT), R29.1, U2.12 (VDD), U2.19 (VDD), U2.27 (VDD), U2.34 (VDD), U2.4 (VDD), U2.42 (VDD), U2.49 (VDD), U2.57 (VDD), U2.61 (VDD), U2.62 (VDD), U2.63 (VDD), U2.64 (VDD)
- new net +0V9_XU_FB: R29.2, R30.1
- new net +1V8_XU: IC10.5 (OUT), U2.17 (VDDIOB18), U2.22 (PLL_AVDD), U2.26 (VDDIOB18), U2.31 (USB_VDD18), U3.18 (V1P8V2_B), U3.24 (VCC2), U3.25 (V1P8V2_A)
- new net XU_QSPI_CS: U2.3 (X0D01_SS), U4.1 (CS#)
- new net XU_QSPI_IO0: U2.59 (X0D04_IO0), U4.5 (DI_IO0)
- new net XU_QSPI_IO1: U2.1 (X0D05), U4.2 (DO_IO1)
- new net XU_QSPI_IO2: U2.60 (X0D06_IO2), U4.7 (HOLD#_IO3)
- new net XU_QSPI_IO3: U2.2 (X0D07), U4.3 (WP#_IO2)
- new net XU_QSPI_SCLK: U2.5 (X0D10_SCLK), U4.6 (CLK)
- new net XU_TCK: JP2.4 (Pin_4), U2.24 (TCK)
- new net XU_TDI: JP2.1 (Pin_1), U2.18 (TDI)
- new net XU_TDO: JP2.2 (Pin_2), U2.20 (TDO)
- new net XU_TMS: JP2.3 (Pin_3), U2.23 (TMS)
- new net XU_USB_DM: U2.28 (USB_DM), U3.22 (DD-)
- new net XU_USB_DP: U2.29 (USB_DP), U3.21 (DD+)
- new net XU_XIN: C34.1, Y1.1
- new net XU_XOUT: C35.1, Y1.2

Commit message: Complete power/decoupling wiring; supersede concurrent layout cleanup
Two independent sessions worked from commit 8e62d29 in parallel, in
separate working copies:

1. A Codex session in this repo (uncommitted) did a pure visual layout
   cleanup of AK4490DAC.kicad_sch/.kicad_sym - regrouped functional
   blocks, fit everything on one page, widened XU316/ISOUSB211 pin
   spacing. Verified electrically identical to 8e62d29 (same 154-net
   netlist, same 135 ERC violations, same symbol UUIDs/properties).
   Left uncommitted; backed up to
   .wiring-cleanup/discarded-layout-backup/ before being superseded by
   this commit, per user decision (wiring completeness prioritized over
   layout aesthetics - the layout can be redone on the finished design
   later). Its own docs kept at docs/WIRING_CLEANUP_RESULT.md.

2. A separate Codex session in a scratch copy of this repo
   (C:\Users\ftomo\Documents\ChatGPT\AK4490DAC) did the actual power
   wiring pass: connected +VIN_RAW -> IC9 (AMS1117) -> +5V5_PRE
   pre-regulator, distributed +5V5_PRE to all 7 downstream LDOs'
   IN/EN/GND, wired their outputs to +3V3_XU/+1V8_XU/+0V9_XU/
   +3V3_4490/+3V3A_4490/+5V_4490_L/+5V_4490_R, wired AK4490's full
   power/reference network (C8-C13), XU316's crystal + reset, and
   ISOUSB211/USB-C NC pins. Fixed duplicate TCM809 references (U3->U8,
   U4->U9) and corrected IC11 from a nonexistent "TPS7A20-ADJ" to the
   real fixed-0.9V TPS7A2009PDBVR. ERC 135 -> 17 violations. Left its
   own handoff at docs/HANDOFF_CLAUDE_WIRING.md.

This commit is Claude's continuation of that second session's work,
still in the ChatGPT scratch copy, now merged into this repo (chosen
over the layout-cleanup copy per user decision, since the two diverged
in incompatible coordinate systems and a coordinate-level merge of both
wasn't practical):

- Removed U1 (SN74LS06N): fully unwired leftover with no other
  reference in the schematic (symbol instance + lib_symbols cache
  entry removed). Fixed missing_unit/mi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
Parts:
- removed R29: 1.2k, Resistor_SMD:R_0603_1608Metric, symbol Device:R
- removed R30: 10k, Resistor_SMD:R_0603_1608Metric, symbol Device:R
- removed U1: SN74LS06NSR, Package_SO:SOIC-14_3.9x8.7mm_P1.27mm, symbol 74xx:74LS06N
- added C36, C39, C40, C41, C42, C43, C44, C45, C46, C47, C48, C49, C50, C51, C52: 1uF, Capacitor_SMD:C_0603_1608Metric, symbol Device:C
- added C37, C38: 0.1uF, Capacitor_SMD:C_0603_1608Metric, symbol Device:C
- added C53, C54: 10uF, Capacitor_SMD:C_0603_1608Metric, symbol Device:C
- IC11: value TPS7A20-ADJ -> TPS7A2009PDBVR
- renumbered U3 to U8, U4 to U9
Connections:
- net +0V9_XU is gone; now on net +3V3A_4490: IC11.5 (OUT), U2.12 (VDD), U2.19 (VDD), U2.27 (VDD), U2.34 (VDD), U2.4 (VDD), U2.42 (VDD), U2.49 (VDD), U2.57 (VDD), U2.61 (VDD), U2.62 (VDD), U2.63 (VDD), U2.64 (VDD)
- net +1V8_XU is gone; now on net +3V3A_4490: IC10.5 (OUT), U2.17 (VDDIOB18), U2.22 (PLL_AVDD), U2.26 (VDDIOB18), U2.31 (USB_VDD18), U3.18 (V1P8V2_B), U3.24 (VCC2), U3.25 (V1P8V2_A)
- net +3V3_118 is gone; now on net +3V3A_4490: C28.1, U8.3 (V_{DD})
- net +3V3_4490 is gone; now on net +3V3A_4490: C29.1, U6.10 (DIF0), U6.11 (DIF1), U6.13 (PSN), U6.15 (DEM0), U6.17 (ACKS), U6.8 (SD), U9.3 (V_{DD})
- net +3V3_XU is gone; now on net +3V3A_4490: IC1.5 (OUT), U2.30 (USB_VDD33), U2.38 (VDDIOR), U2.52 (VDDIOT), U2.8 (VDDIOL), U3.16 (CDPENZ2), U3.27 (V3P3V2), U3.28 (VBUS2), U4.8 (VCC)
- net +VIN_RAW is gone; now on net +3V3A_4490: J1.1 (Pin_1), U7.2 (+Vin)
- net GND is gone; now on net +3V3A_4490: C24.2, C28.2, C29.2, C32.2, C34.2, C35.2, IC1.2 (GND), IC10.2 (GND), IC11.2 (GND), J1.2 (Pin_2), J4.2 (Pin_2), J5.2 (Pin_2), JP2.5 (Pin_5), R16.2, R23.2, R25.2, R26.2, U2.65 (VSS_EP), U3.17 (GND2_B), U3.19 (EQ21), U3.20 (EQ20), U3.26 (GND2), U4.4 (GND), U6.1 (NC1), U6.12 (DIF2), U6.14 (I2C), U6.16 (DEM1), U6.18 (NC18), U6.21 (VREFLR), U6.22 (VREFLR*), U6.24 (NC24), U6.37 (NC37), U6.39 (VREFLL), U6.40 (VREFLL*), U6.43 (NC43), U6.6 (SSLOW), U6.7 (SMUTE), U6.9 (SLOW), U7.1 (-Vin), U7.3 (CON), U7.7 (Common), U8.1 (GND), U9.1 (GND)
- net RST_118 is gone; now on net XU_RST_N: R25.1, U8.2 (~{RESET})
- net +3V3A_4490: now also C10.1, C10.2, C11.1, C11.2, C12.1, C12.2, C13.1, C13.2, C8.2, C9.2, IC1.1 (IN), IC1.3 (EN), IC10.1 (IN), IC10.3 (EN), IC11.1 (IN), IC11.3 (EN), IC2.1 (IN), IC2.2 (GND), IC2.3 (EN), IC2.5 (OUT), IC3.1 (IN), IC3.2 (GND), IC3.3 (EN), IC3.5 (OUT), IC4.1 (IN), IC4.2 (GND), IC4.3 (EN), IC4.5 (OUT), IC8.1 (IN), IC8.2 (GND), IC8.3 (EN), IC8.5 (OUT), IC9.2 (VO), IC9.3 (VI), R3.2, R4.1, U6.27 (VDDR), U6.28 (VDDR*), U6.29 (VSSR), U6.30 (VSSR*), U6.31 (VSSL), U6.32 (VSSL*), U6.33 (VDDL), U6.34 (VDDL*), U6.44 (AVDD), U6.45 (AVSS), U6.47 (DVSS), U6.48 (DVDD), C39.1, C39.2, C40.1, C40.2, C41.1, C41.2, C42.1, C42.2, C43.1, C43.2, C44.1, C44.2, C45.1, C45.2, C46.1, C46.2, C47.1, C47.2, C48.1, C48.2, C49.1, C49.2, C50.1, C50.2, C51.1, C51.2, C52.1, C52.2, C53.1, C53.2, C54.1, C54.2
- net USB_GND: now also C36.2, C37.2, C38.2
- net XU_XIN: now also U2.16 (XIN)
- net XU_XOUT: now also U2.15 (XOUT)
- net XU_RST_N: now reaches U2.21 (RST_N)
- net at IC9.1 (ADJ): now also R3.1, R4.2
- net at U3.11 (V1P8V1_B): now also C38.1
- net at U3.2 (V3P3V1): now also C36.1
- net at U3.4 (V1P8V1_A): now also C37.1
- net VCMR: now reaches U6.23 (VCMR)
- net VCMR: now also C8.1
- net VCML: now reaches U6.38 (VCML)
- net VCML: now also C9.1
- no-connect marks 0 -> 28
Other:
- note added: "01 USB-C INPUT"
- note added: "02 USB ISOLATION"
- note added: "03 XMOS / USB AUDIO"
- note added: "04 DAC / REFERENCES"
- note added: "05 LEFT ANALOG OUTPUT"
- note added: "06 RIGHT ANALOG OUTPUT"
- note added: "07 POWER SUPPLIES"
- note added: "24 MHz CLOCK"
- note added: "AK4490 USB DAC"
- note added: "AK4490 | digital control / analog reference"
- note added: "AUXILIARY LOGIC"
- note added: "DC input / digital rails / DAC rails / analog +/-15 V"
- note added: "Differential input > filter / MUSES8920 > LINE_OUT_L"
- note added: "Differential input > filter / MUSES8920 > LINE_OUT_R"
- note added: "I2S GPIO assignments are provisional."
- note added: "ISOUSB211 | USB_GND <-> main GND"
- note added: "Isolation domains are retained."
- note added: "JTAG DEBUG"
- note added: "OP-AMP SUPPLY"
- note added: "PC / USB bus power / USB_GND"
- note added: "Power rails connected; regulator bypass capacitors still required."
- note added: "QSPI BOOT FLASH"
- note added: "REFERENCE BYPASS"
- note added: "RESET SUPERVISORS"
- note added: "Reset supervisors renumbered U8 / U9."
- note added: "SIGNAL FLOW USB INPUT > ISOLATION > XMOS / I2S > DAC > ANALOG FILTER / LINE OUTPUT"
- note added: "USB signals connect by matching net labels."
- note added: "XU316 | I2S / QSPI boot / clock / debug"
- title: AK4490DAC -> AK4490 USB DAC - functional layout
- moved on the sheet: C10, C11, C12, C13, C22, C23, C24, C25, C26, C27, C28, C29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
